Commit message: finished the migration of the car:poop:

File: src/simulation/urdf/gazebo/kinect.xacro (robot description, xacro)
@@ -16,5 +16,5 @@
           </clip>
         </camera>
-        <plugin name="kinect_camera_controller" filename="libgazebo_ros_openni_kinect.so">
+        <!-- <plugin name="kinect_camera_controller" filename="libgazebo_ros_openni_kinect.so">
           <cameraName>camera</cameraName>
           <alwaysOn>true</alwaysOn>
@@ -33,4 +33,28 @@
           <distortion_t2>0.0</distortion_t2>
           <pointCloudCutoff>0.4</pointCloudCutoff>
+        </plugin> -->
+        <plugin name="plugin_name_whatever" filename="libgazebo_ros_camera.so">
+            <!-- Change namespace, camera name and topics so -
+              * Raw images are published to: /custom_ns/custom_camera/custom_image
+              * Depth images are published to: /custom_ns/custom_camera/custom_image_depth
+              * Raw image camera info is published to: /custom_ns/custom_camera/custom_info_raw
+              * Depth image camera info is published to: /custom_ns/custom_camera/custom_info_depth
+              * Point cloud is published to: /custom_ns/custom_camera/custom_points
+        -->
+            <ros>
+                <namespace>camera</namespace>
+                <remapping>custom_camera/image_raw:=custom_camera/custom_image</remapping>
+                <remapping>custom_camera/image_depth:=custom_camera/custom_image_depth</remapping>
+                <remapping>custom_camera/camera_info:=custom_camera/custom_info_raw</remapping>
+                <remapping>custom_camera/camera_info_depth:=custom_camera/custom_info_depth</remapping>
+                <remapping>custom_camera/points:=custom_camera/custom_points</remapping>
+            </ros>
+            <!-- Set camera name. If empty, defaults to sensor name (i.e. "sensor_name") -->
+            <camera_name>custom_camera</camera_name>
+            <!-- Set TF frame name. If empty, defaults to link name (i.e. "link_name") -->
+            <frame_name>link_camera_fake</frame_name>
+            <hack_baseline>0.07</hack_baseline>
+            <!-- No need to repeat distortion parameters or to set autoDistortion -->
+            <min_depth>0.001</min_depth>
         </plugin>
       </sensor>

File: src/simulation/urdf/gazebo/laser.xacro (robot description, xacro)
@@ -26,7 +26,9 @@
         </noise>
       </ray>
-      <plugin name="gazebo_rplidar" filename="libgazebo_ros_laser.so">
-        <topicName>/scan</topicName>
-        <frameName>laser</frameName>
+      <plugin name="gazebo_ros_head_hokuyo_controlle" filename="libgazebo_ros_ray_sensor.so" >
+        <ros>
+          <remapping>~/out:=/scan</remapping>
+        </ros>
+        <output_type>sensor_msgs/LaserScan</output_type>
       </plugin>
     </sensor>

File: src/simulation/urdf/gazebo/move.xacro (robot description, xacro)
@@ -22,5 +22,4 @@
   </ros2_control>
   <gazebo>
-    <!-- Joint state publisher -->
     <plugin filename="libgazebo_ros2_control.so" name="gazebo_ros2_control">
       <parameters>$(find simulation)/param/diff_drive_controller.yaml</parameters>

File: src/simulation/urdf/xacro/car.urdf.xacro (robot description, xacro)
@@ -7,5 +7,5 @@
     <xacro:include filename="../gazebo/move.xacro" />
     <xacro:include filename="../gazebo/laser.xacro" />
-    <xacro:include filename="../gazebo/camera.xacro" />
+    <!-- <xacro:include filename="../gazebo/camera.xacro" /> -->
     <xacro:include filename="../gazebo/kinect.xacro" />
 </robot>

File: src/simulation/urdf/xacro/car_base.urdf.xacro (robot description, xacro)
@@ -46,5 +46,5 @@
     <!-- qudong wheel -->
     <xacro:property name="wheel_radius" value="0.0325" />
-    <xacro:property name="wheel_length" value="0.015" />
+    <xacro:property name="wheel_length" value="0.05" />
     <xacro:property name="wheel_mass" value="0.05" />
     <xacro:macro name="add_wheels" params="name flag">
