Commit message: :fire:

File: src/simulation/urdf/xacro/car_base.urdf.xacro (robot description, xacro)
@@ -46,5 +46,5 @@
     <!-- qudong wheel -->
     <xacro:property name="wheel_radius" value="0.0325" />
-    <xacro:property name="wheel_length" value="0.05" />
+    <xacro:property name="wheel_length" value="0.015" />
     <xacro:property name="wheel_mass" value="0.05" />
     <xacro:macro name="add_wheels" params="name flag">
